File: kicad/playboyzinho.kicad_sch (KiCad schematic)
At the start: 17 parts, among them SW1 SW_Push, SW2 SW_Push, SW3 SW_Push, SW4 SW_Push, SW5 SW_Push, SW6 SW_Push, SW7 SW_Push, SW8 SW_Push, SW9 SW_SPDT, U1 esp32-s3-pl, U7 (amplificador)_MAX98357_Module

Commit message: refact: separa conexões SD da tela e adiciona uma conexão ao SD do amplificador
Connections:
- net SD_CS: now also U1.7 (GPIO7); no longer U1.4 (GPIO4)
- net TFT_MOSI: now reaches U1.11 (GPIO18)
- net TFT_MOSI: now also U4.6 (SDI-(MOSI))
- net SD_MISO: now reaches U1.5 (GPIO5)
- net SD_MISO: now also U4.17 (SD_MISO)
- net SD_MOSI: now reaches U1.6 (GPIO6)
- net SD_MOSI: now also U4.16 (SD_MOSI)
- net TFT_SCK: now reaches U1.8 (GPIO15)
- net TFT_SCK: now also U4.7 (SCK)
- net AMP_SD: now reaches U7.5 (SD)
- net AMP_SD: now also U1.17 (GPIO11)
- net CS renamed TFT_CS
- net TFT_CS: now also U1.16 (GPIO10); no longer U1.17 (GPIO11)
- net DC renamed TFT_DC
- net TFT_DC: now also U1.12 (GPIO8); no longer U1.15 (GPIO9)
- net MISO renamed TFT_MISO
- net TFT_MISO: no longer U4.17 (SD_MISO)
- removed net MOSI: U1.12 (GPIO8), U4.16 (SD_MOSI), U4.6 (SDI-(MOSI))
- net RESET renamed TFT_RESET
- net TFT_RESET: now also U1.15 (GPIO9); no longer U1.16 (GPIO10)
- removed net SCK: U1.10 (GPIO17), U4.18 (SD_SCK), U4.7 (SCK)
- new net SD_SCK: U1.4 (GPIO4), U4.18 (SD_SCK)
- no-connect marks 32 -> 27

Commit message: refact: tira sd do amplificador do GPIO11 e coloca num SPDT
Parts:
- added SW10: SW_SPDT, lib-do-playboy:alavanca, symbol Switch:SW_SPDT
Connections:
- net 3V3: now also SW10.3 (C)
- net AMP_SD: now also SW10.2 (B); no longer U1.17 (GPIO11)
- net Button-1: now also U1.27 (GPIO2); no longer U1.28 (GPIO42)
- net Button-2: now also U1.28 (GPIO42); no longer U1.29 (GPIO41)
- net Button-3: now also U1.29 (GPIO41); no longer U1.30 (GPIO40)
- net Button-4: now also U1.31 (GPIO39); no longer U1.32 (GPIO38)
- net Button-5: now also U1.30 (GPIO40); no longer U1.31 (GPIO39)
- net Button-6: now also U1.32 (GPIO38); no longer U1.38 (GPIO48)
- net GND: now also SW10.1 (A)
- no-connect marks 27 -> 28
Other:
- moved on the sheet: U3, U7
